Commit message: Cambio de nombre, mapas agregados

File: urdf/rover.urdf.xacro (robot description, xacro)
@@ -1,4 +1,4 @@
 <?xml version="1.0" encoding="utf-8"?>
-<robot name="rover_RYCSV" xmlns:xacro="http://ros.org/wiki/xacro">
+<robot name="rover" xmlns:xacro="http://ros.org/wiki/xacro">
   <xacro:arg name="imu_enable" default="true"/>
   <xacro:arg name="gps_enable" default="true"/>
@@ -29,5 +29,5 @@
       <geometry>
         <mesh
-          filename="package://rover_RYCSV/meshes/Caja.STL" />
+          filename="package://rover/meshes/Caja.STL" />
       </geometry>
       <material
@@ -42,6 +42,5 @@
         rpy="0 0 0" />
       <geometry>
-        <mesh
-          filename="package://rover_RYCSV/meshes/Caja.STL" />
+        <box size="0.01 0.05 0.05"/>
       </geometry>
     </collision>
@@ -82,5 +81,5 @@
       <geometry>
         <mesh
-          filename="package://rover_RYCSV/meshes/Rocker_izq.STL" />
+          filename="package://rover/meshes/Rocker_izq.STL" />
       </geometry>
       <material
@@ -95,6 +94,5 @@
         rpy="0 0 0" />
       <geometry>
-        <mesh
-          filename="package://rover_RYCSV/meshes/Rocker_izq.STL" />
+        <box size="0.01 0.05 0.05"/>
       </geometry>
     </collision>
@@ -137,5 +135,5 @@
       <geometry>
         <mesh
-          filename="package://rover_RYCSV/meshes/Bogie_izq.STL" />
+          filename="package://rover/meshes/Bogie_izq.STL" />
       </geometry>
       <material
@@ -150,6 +148,5 @@
         rpy="0 0 0" />
       <geometry>
-        <mesh
-          filename="package://rover_RYCSV/meshes/Bogie_izq.STL" />
+        <box size="0.01 0.05 0.05"/>
       </geometry>
     </collision>
@@ -192,5 +189,5 @@
       <geometry>
         <mesh
-          filename="package://rover_RYCSV/meshes/Acople_1.STL" />
+          filename="package://rover/meshes/Acople_1.STL" />
       </geometry>
       <material
@@ -205,6 +202,5 @@
         rpy="0 0 0" />
       <geometry>
-        <mesh
-          filename="package://rover_RYCSV/meshes/Acople_1.STL" />
+        <box size="0.01 0.05 0.05"/>
       </geometry>
     </collision>
@@ -247,5 +243,5 @@
       <geometry>
         <mesh
-          filename="package://rover_RYCSV/meshes/Rueda_1.STL" />
+          filename="package://rover/meshes/Rueda_1.STL" />
       </geometry>
       <material
@@ -261,5 +257,5 @@
       <geometry>
         <mesh
-          filename="package://rover_RYCSV/meshes/Rueda_1.STL" />
+          filename="package://rover/meshes/Rueda_1.STL" />
       </geometry>
     </collision>
@@ -303,5 +299,5 @@
       <geometry>
         <mesh
-          filename="package://rover_RYCSV/meshes/Acople_2.STL" />
+          filename="package://rover/meshes/Acople_2.STL" />
       </geometry>
       <material
@@ -316,6 +312,5 @@
         rpy="0 0 0" />
       <geometry>
-        <mesh
-          filename="package://rover_RYCSV/meshes/Acople_2.STL" />
+        <box size="0.01 0.05 0.05"/>
       </geometry>
     </collision>
@@ -356,5 +351,5 @@
       <geometry>
         <mesh
-          filename="package://rover_RYCSV/meshes/Rueda_2.STL" />
+          filename="package://rover/meshes/Rueda_2.STL" />
       </geometry>
       <material
@@ -370,5 +365,5 @@
       <geometry>
         <mesh
-          filename="package://rover_RYCSV/meshes/Rueda_2.STL" />
+          filename="package://rover/meshes/Rueda_2.STL" />
       </geometry>
     </collision>
@@ -412,5 +407,5 @@
       <geometry>
         <mesh
-          filename="package://rover_RYCSV/meshes/Acople_3.STL" />
+          filename="package://rover/meshes/Acople_3.STL" />
       </geometry>
       <material
@@ -425,6 +420,5 @@
         rpy="0 0 0" />
       <geometry>
-        <mesh
-          filename="package://rover_RYCSV/meshes/Acople_3.STL" />
+        <box size="0.01 0.05 0.05"/>
       </geometry>
     </collision>
@@ -467,5 +461,5 @@
       <geometry>
         <mesh
-          filename="package://rover_RYCSV/meshes/Rueda_3.STL" />
+          filename="package://rover/meshes/Rueda_3.STL" />
       </geometry>
       <material
@@ -481,5 +475,5 @@
       <geometry>
         <mesh
-          filename="package://rover_RYCSV/meshes/Rueda_3.STL" />
+          filename="package://rover/meshes/Rueda_3.STL" />
       </geometry>
     </collision>
@@ -523,5 +517,5 @@
       <geometry>
         <mesh
-          filename="package://rover_RYCSV/meshes/Rocker_der.STL" />
+          filename="package://rover/meshes/Rocker_der.STL" />
       </geometry>
       <material
@@ -536,6 +530,5 @@
         rpy="0 0 0" />
       <geometry>
-        <mesh
-          filename="package://rover_RYCSV/meshes/Rocker_der.STL" />
+        <box size="0.01 0.05 0.05"/>
       </geometry>
     </collision>
@@ -578,5 +571,5 @@
       <geometry>
         <mesh
-          filename="package://rover_RYCSV/meshes/Bogie_der.STL" />
+          filename="package://rover/meshes/Bogie_der.STL" />
       </geometry>
       <material
@@ -591,6 +584,5 @@
         rpy="0 0 0" />
       <geometry>
-        <mesh
-          filename="package://rover_RYCSV/meshes/Bogie_der.STL" />
+        <box size="0.01 0.05 0.05"/>
       </geometry>
     </collision>
@@ -633,5 +625,5 @@
       <geometry>
         <mesh
-          filename="package://rover_RYCSV/meshes/Acople_4.STL" />
+          filename="package://rover/meshes/Acople_4.STL" />
       </geometry>
       <material
@@ -646,6 +638,5 @@
         rpy="0 0 0" />
       <geometry>
-        <mesh
-          filename="package://rover_RYCSV/meshes/Acople_4.STL" />
+        <box size="0.01 0.05 0.05"/>
       </geometry>
     </collision>
@@ -688,5 +679,5 @@
       <geometry>
         <mesh
-          filename="package://rover_RYCSV/meshes/Rueda_4.STL" />
+          filename="package://rover/meshes/Rueda_4.STL" />
       </geometry>
       <material
@@ -702,5 +693,5 @@
       <geometry>
         <mesh
-          filename="package://rover_RYCSV/meshes/Rueda_4.STL" />
+          filename="package://rover/meshes/Rueda_4.STL" />
       </geometry>
     </collision>
@@ -744,5 +735,5 @@
       <geometry>
         <mesh
-          filename="package://rover_RYCSV/meshes/Acople_5.STL" />
+          filename="package://rover/meshes/Acople_5.STL" />
       </geometry>
       <material
@@ -757,6 +748,5 @@
         rpy="0 0 0" />
       <geometry>
-        <mesh
-          filename="package://rover_RYCSV/meshes/Acople_5.STL" />
+        <box size="0.01 0.05 0.05"/>
       </geometry>
     </collision>
@@ -797,5 +787,5 @@
       <geometry>
         <mesh
-          filename="package://rover_RYCSV/meshes/Rueda_5.STL" />
+          filename="package://rover/meshes/Rueda_5.STL" />
       </geometry>
       <material
@@ -811,5 +801,5 @@
       <geometry>
         <mesh
-          filename="package://rover_RYCSV/meshes/Rueda_5.STL" />
+          filename="package://rover/meshes/Rueda_5.STL" />
       </geometry>
     </collision>
@@ -853,5 +843,5 @@
       <geometry>
         <mesh
-          filename="package://rover_RYCSV/meshes/Acople_6.STL" />
+          filename="package://rover/meshes/Acople_6.STL" />
       </geometry>
       <material
@@ -866,6 +856,5 @@
         rpy="0 0 0" />
       <geometry>
-        <mesh
-          filename="package://rover_RYCSV/meshes/Acople_6.STL" />
+        <box size="0.01 0.05 0.05"/>
       </geometry>
     </collision>
@@ -908,5 +897,5 @@
       <geometry>
         <mesh
-          filename="package://rover_RYCSV/meshes/Rueda_6.STL" />
+          filename="package://rover/meshes/Rueda_6.STL" />
       </geometry>
       <material
@@ -922,5 +911,5 @@
       <geometry>
         <mesh
-          filename="package://rover_RYCSV/meshes/Rueda_6.STL" />
+          filename="package://rover/meshes/Rueda_6.STL" />
       </geometry>
     </collision>
@@ -1081,5 +1070,5 @@
   <!-- SENSOR KINECT -->
   <xacro:if value="$(arg kinect_enable)">
-    <xacro:include filename="$(find rover_RYCSV)/urdf/kinect.gazebo.xacro" />
+    <xacro:include filename="$(find rover)/urdf/kinect.gazebo.xacro" />
     <link name="Sensor_kinect">
       <inertial>
@@ -1103,5 +1092,5 @@
         <geometry>
           <mesh
-            filename="package://rover_RYCSV/meshes/sensor_kinect.stl"
+            filename="package://rover/meshes/sensor_kinect.stl"
             scale= "0.01 0.01 0.01"/>
         </geometry>
@@ -1118,5 +1107,5 @@
         <geometry>
           <mesh
-            filename="package://rover_RYCSV/meshes/sensor_kinect.stl"
+            filename="package://rover/meshes/sensor_kinect.stl"
             scale= "0.01 0.01 0.01"/>
         </geometry>
@@ -1151,6 +1140,6 @@
   <!-- CAMARA Y LIDAR -->
   <xacro:if value="$(arg camera_and_lidar_enable)">
-    <xacro:include filename="$(find rover_RYCSV)/urdf/camera.gazebo.xacro" />
-    <xacro:include filename="$(find rover_RYCSV)/urdf/lidar.gazebo.xacro" />
+    <xacro:include filename="$(find rover)/urdf/camera.gazebo.xacro" />
+    <xacro:include filename="$(find rover)/urdf/lidar.gazebo.xacro" />
     <link name="Camera">
       <inertial>
@@ -1213,5 +1202,5 @@
         <origin xyz="0 0 0" rpy="0 0 0"/>
         <geometry>
-          <mesh filename="package://rover_RYCSV/meshes/hokuyo.dae"/>
+          <mesh filename="package://rover/meshes/hokuyo.dae"/>
         </geometry>
       </visual>
@@ -1238,5 +1227,5 @@
   <!-- SENSOR IMU -->
   <xacro:if value="$(arg imu_enable)">
-    <xacro:include filename="$(find rover_RYCSV)/urdf/imu.gazebo.xacro" />
+    <xacro:include filename="$(find rover)/urdf/imu.gazebo.xacro" />
     <link name="IMU">
       <inertial>
@@ -1291,5 +1280,5 @@
   </xacro:if>
   <xacro:if value="$(arg gps_enable)">
-    <xacro:include filename="$(find rover_RYCSV)/urdf/gps.gazebo.xacro" />
+    <xacro:include filename="$(find rover)/urdf/gps.gazebo.xacro" />
     <link name="GPS">
       <inertial>
